File: CH341Apro.sch (KiCad schematic (older format))
At the start: 18 parts, among them J1 USB_A, J2 Conn_01x07, J3 ZIF-16, J4 Conn_01x07, U1 AMS1117-3.3, U2 CH341a, U3 SPI FLASH, U4 I2C EEPROM, Y1 12M

Commit message: Updated schematic and PCB
Read the README file for details
Parts:
- removed C4: 472, Capacitor_SMD:C_0603_1608Metric, symbol Device:C
- removed J2, J4: Conn_01x07, Connector_PinSocket_2.54mm:PinSocket_1x07_P2.54mm_Vertical, symbol Connector_Generic:Conn_01x07
- removed U3: SPI FLASH, Package_SO:SOIC-16W_7.5x10.3mm_P1.27mm, symbol Memory_Flash:IS25WP256D-xM
- removed U4: I2C EEPROM, Package_SO:SOIC-8_3.9x4.9mm_P1.27mm, symbol Memory_EEPROM:M24C01-FMN
- added C3: 472, Capacitor_SMD:C_0603_1608Metric, symbol Device:C
- added J4: (no value), Connector_PinHeader_2.54mm:PinHeader_1x09_P2.54mm_Vertical, symbol Connector_Generic:Conn_01x09
- added J5: V_SEL, Connector_PinHeader_2.54mm:PinHeader_1x03_P2.54mm_Vertical, symbol Connector_Generic:Conn_01x03
- added R2: 0R, Resistor_SMD:R_0805_2012Metric, symbol Device:R
- J1: footprint connectors:USB_A_MALE_Generic -> Connector_USB:USB_A_CNCTech_1001-011-01101_Horizontal; symbol Connector:USB_A -> CH341Apro-rescue:USB_A-Connector
- Y1: footprint Crystal:Crystal_HC49-U_Vertical -> Crystal:Crystal_HC49-4H_Vertical
Connections:
- net labels added: USB_N, USB_P, VCC
- net labels removed: 1, 2, 3, RXD, TXD
- wire segments 141 -> 145
Other:
- moved on the sheet: C1, C2, J3, U1

Commit message: Add JLCPCB assembly infos
Parts:
- removed R2: 0R, Resistor_SMD:R_0805_2012Metric, symbol Device:R
- added JP1: (no value), Jumper:SolderJumper-2_P1.3mm_Open_Pad1.0x1.5mm, symbol Jumper:SolderJumper_2_Open
- C1, C2: LCSC (none) -> C19702
- C3: LCSC (none) -> C8032
- C5, C6: footprint Capacitor_SMD:C_0603_1608Metric -> Capacitor_SMD:C_0402_1005Metric; LCSC (none) -> C1554
- D1: value Power -> PWR; LCSC (none) -> C72044
- D2: LCSC (none) -> C72043
- J1: symbol CH341Apro-rescue:USB_A-Connector -> CH341Apro-rescue:USB_A-Connector-CH341Apro-rescue
- R1: footprint Resistor_SMD:R_0805_2012Metric -> Resistor_SMD:R_0603_1608Metric; LCSC (none) -> C207010
- RN1: LCSC (none) -> C12001
- U1: LCSC (none) -> C351784
- U2: LCSC (none) -> C13517
- Y1: footprint Crystal:Crystal_HC49-4H_Vertical -> Crystal:Crystal_SMD_5032-2Pin_5.0x3.2mm; LCSC (none) -> C112573
Connections:
- net 3V3: now also JP1.2 (B)
- net at C3.2, U2.9 (V3): now also JP1.1 (A)
Changed lines of the file:
@@
 F 2 "Package_TO_SOT_SMD:SOT-223-3_TabPin2" H 2950 1250 50  0001 C CNN
 F 3 "http://www.advanced-monolithic.com/pdf/ds1117.pdf" H 3050 800 50  0001 C CNN
+F 4 "C351784" H 2950 1050 50  0001 C CNN "LCSC"
 	1    2950 1050
 	1    0    0    -1
@@
 F 0 "R1" H 1150 1550 50  0000 L CNN
 F 1 "0R" H 1150 1450 50  0000 L CNN
-F 2 "Resistor_SMD:R_0805_2012Metric" V 1280 1500 50  0001 C CNN
+F 2 "Resistor_SMD:R_0603_1608Metric" V 1280 1500 50  0001 C CNN
 F 3 "~" H 1350 1500 50  0001 C CNN
+F 4 "C207010" H 1350 1500 50  0001 C CNN "LCSC"
 	1    1350 1500
 	1    0    0    -1
@@
 F 2 "Resistor_SMD:R_Array_Convex_4x0603" V 5920 2100 50  0001 C CNN
 F 3 "~" H 6000 2100 50  0001 C CNN
+F 4 "C12001" H 6000 2100 50  0001 C CNN "LCSC"
 	1    6000 2100
 	1    0    0    -1
@@
 F 2 "Resistor_SMD:R_Array_Convex_4x0603" V 5770 1800 50  0001 C CNN
 F 3 "~" H 5850 1800 50  0001 C CNN
+F 4 "C12001" H 5850 1800 50  0001 C CNN "LCSC"
 	2    5850 1800
 	1    0    0    -1
@@
 F 2 "Resistor_SMD:R_Array_Convex_4x0603" V 1620 1100 50  0001 C CNN
 F 3 "~" H 1700 1100 50  0001 C CNN
+F 4 "C12001" H 1700 1100 50  0001 C CNN "LCSC"
 	3    1700 1100
 	1    0    0    -1
@@
 F 2 "Resistor_SMD:R_Array_Convex_4x0603" V 2720 1900 50  0001 C CNN
 F 3 "~" H 2800 1900 50  0001 C CNN
+F 4 "C12001" V 2800 1900 50  0001 C CNN "LCSC"
 	4    2800 1900
 	0    -1   -1   0
@@
 F 2 "Capacitor_SMD:C_0603_1608Metric" H 2488 1150 50  0001 C CNN
 F 3 "~" H 2450 1300 50  0001 C CNN
+F 4 "C19702" H 2450 1300 50  0001 C CNN "LCSC"
 	1    2450 1300
 	1    0    0    -1
@@
 F 2 "LED_SMD:LED_0603_1608Metric" H 5950 1250 50  0001 C CNN
 F 3 "~" H 5950 1250 50  0001 C CNN
+F 4 "C72043" V 5950 1250 50  0001 C CNN "LCSC"
 	1    5950 1250
 	0    -1   -1   0
@@
 P 1700 1500
 F 0 "D1" V 1739 1382 50  0000 R CNN
-F 1 "Power" V 1650 1350 50  0000 R CNN
+F 1 "PWR" V 1650 1350 50  0000 R CNN
 F 2 "LED_SMD:LED_0603_1608Metric" H 1700 1500 50  0001 C CNN
 F 3 "~" H 1700 1500 50  0001 C CNN
+F 4 "C72044" V 1700 1500 50  0001 C CNN "LCSC"
 	1    1700 1500
 	0    -1   -1   0
@@
 F 2 "Capacitor_SMD:C_0603_1608Metric" H 3488 1150 50  0001 C CNN
 F 3 "~" H 3450 1300 50  0001 C CNN
+F 4 "C19702" H 3450 1300 50  0001 C CNN "LCSC"
 	1    3450 1300
 	1    0    0    -1
@@
 F 0 "Y1" H 2800 3818 50  0000 C CNN
 F 1 "12M" H 2800 3727 50  0000 C CNN
-F 2 "Crystal:Crystal_HC49-4H_Vertical" H 2800 3550 50  0001 C CNN
+F 2 "Crystal:Crystal_SMD_5032-2Pin_5.0x3.2mm" H 2800 3550 50  0001 C CNN
 F 3 "~" H 2800 3550 50  0001 C CNN
+F 4 "C112573" H 2800 3550 50  0001 C CNN "LCSC"
 	1    2800 3550
 	1    0    0    -1
@@
 F 0 "C5" H 2715 3946 50  0000 L CNN
 F 1 "20p" H 2715 3855 50  0000 L CNN
-F 2 "Capacitor_SMD:C_0603_1608Metric" H 2638 3750 50  0001 C CNN
+F 2 "Capacitor_SMD:C_0402_1005Metric" H 2638 3750 50  0001 C CNN
 F 3 "~" H 2600 3900 50  0001 C CNN
+F 4 "C1554" H 2600 3900 50  0001 C CNN "LCSC"
 	1    2600 3900
 	1    0    0    -1
@@
 F 0 "C6" H 3115 3946 50  0000 L CNN
 F 1 "20p" H 3115 3855 50  0000 L CNN
-F 2 "Capacitor_SMD:C_0603_1608Metric" H 3038 3750 50  0001 C CNN
+F 2 "Capacitor_SMD:C_0402_1005Metric" H 3038 3750 50  0001 C CNN
 F 3 "~" H 3000 3900 50  0001 C CNN
+F 4 "C1554" H 3000 3900 50  0001 C CNN "LCSC"
 	1    3000 3900
 	1    0    0    -1
@@
 GND
 $Comp
-L CH341Apro-rescue:USB_A-Connector J1
+L CH341Apro-rescue:USB_A-Connector-CH341Apro-rescue J1
 U 1 1 5F58AEC8
 P 850 2150
@@
 F 2 "Package_SO:SOIC-28W_7.5x17.9mm_P1.27mm" H 3500 2700 50  0001 C CNN
 F 3 "" H 3500 2700 50  0001 C CNN
+F 4 "C13517" H 3900 2550 50  0001 C CNN "LCSC"
 	1    3900 2550
 	1    0    0    -1
@@
 USB_N
 $Comp
-L Device:R R2
-U 1 1 604EF0F1
-P 2900 2300
-F 0 "R2" H 2700 2350 50  0000 L CNN
-F 1 "0R" H 2700 2250 50  0000 L CNN
-F 2 "Resistor_SMD:R_0805_2012Metric" V 2830 2300 50  0001 C CNN
-F 3 "~" H 2900 2300 50  0001 C CNN
-	1    2900 2300
-	1    0    0    -1
-$EndComp
-$Comp
 L Device:C C3
 U 1 1 604EFB0A
@@
 F 2 "Capacitor_SMD:C_0603_1608Metric" H 2738 2450 50  0001 C CNN
 F 3 "~" H 2700 2600 50  0001 C CNN
+F 4 "C8032" V 2700 2600 50  0001 C CNN "LCSC"
 	1    2700 2600
 	0    -1   -1   0
@@
 Wire Wire Line
 	2900 2100 2750 2100
+$Comp
+L Jumper:SolderJumper_2_Open JP1
+U 1 1 603A2DA5
+P 2900 2300
+F 0 "JP1" V 3000 2450 50  0000 R CNN
+F 1 " " V 2855 2212 50  0000 R CNN
+F 2 "Jumper:SolderJumper-2_P1.3mm_Open_Pad1.0x1.5mm" H 2900 2300 50  0001 C CNN
+F 3 "~" H 2900 2300 50  0001 C CNN
+	1    2900 2300
+	0    -1   -1   0
+$EndComp
 $EndSCHEMATC
